File: main_board.sch (EAGLE design)
At the start: 8 parts, among them U1 MAX9019EKA+T

Commit message: working on the solar circuit
Parts:
- added C2: 10uF, MF_Passives:CAPACITOR_NP_0603
- added C3: 22uF, MF_Passives:CAPACITOR_NP_0603
- added J1: TBL009-254-02GY-2GY, PP_Connectors:CON_01X02_TBL009-254-02GY-2GY
- added L1: 10uH, PP_Passives:INDUCTORLPS4012
- added R10, R7, R8, R9: (no value), MF_Passives:RESISTOR_0805
- added U2: AEM10941-QFN, PP_PowerIC:AEM10941
Connections:
- new net BOOST: C3.P$1, U2.BOOST
- new net BUFSRC: C2.P$1, L1.P$2, U2.BUFSRC
- new net SET_CHRDY: R8.P$2, R9.P$1, U2.SET_CHRDY
- new net SET_OVCH: R10.P$1, R9.P$2, U2.SET_OVCH
- new net SET_OVDIS: R7.P$2, R8.P$1, U2.SET_OVDIS
- new net SOLAR_+V: J1.PIN1, U2.FB_COLD, U2.SRC
- new net SWBOOST: L1.P$1, U2.SWBOOST
- new net VBOOST: R7.P$1
- net GND: now also C2.P$2, C3.P$2, J1.PIN2, R10.P$2

Commit message: AEM10941 circuit complete
Parts:
- added C4, C5, C6: 10uF, MF_Passives:CAPACITOR_NP_0603
- added C7, C8: 10F 3.8V, PP_Passives:CAPACITOR_POLARIZED_12.5MM_PTH
- added J2, J3, J4: 709176001501006, PP_Connectors:CON_01X01_709176001501006
- added L2: 10uH, PP_Passives:INDUCTOR_0603
- added R11, R12, R13, R14, R15, R16, R17, R18, R19, R20, R21, R22, R23, R24, R25, R26: (no value), MF_Passives:RESISTOR_0805
Connections:
- removed net BOOST: C3.P$1, U2.BOOST
- new net BAL: C7.NEG, C8.POS, U2.BAL
- new net BATT: C7.POS, U2.BATT
- new net CFG[0]: R15.P$1, R16.P$2, U2.CFG[0]
- new net CFG[1]: R13.P$1, R14.P$2, U2.CFG[1]
- new net CFG[2]: R11.P$1, R12.P$2, U2.CFG[2]
- new net ENHV: R21.P$1, R22.P$2, U2.ENHV
- new net ENLV: R23.P$1, R24.P$2, U2.ENLV
- new net FB_HV: R25.P$1, R26.P$2, U2.FB_HV
- new net HVOUT: C6.P$1, R25.P$2, U2.HVOUT
- new net LVOUT: C5.P$1, U2.LVOUT
- new net SELMPP[0]: R19.P$1, R20.P$2, U2.SELMPP[0]
- new net SELMPP[1]: R17.P$1, R18.P$2, U2.SELMPP[1]
- new net STATUS[0]: J4.PIN1, U2.STATUS[0]
- new net STATUS[1]: J3.PIN1, U2.STATUS[1]
- new net STATUS[2]: J2.PIN1, U2.STATUS[2]
- new net SWBUCK: L2.P$1, U2.SWBUCK
- new net VBUCK: C4.P$1, L2.P$2, R11.P$2, R13.P$2, R15.P$2, R17.P$2, R19.P$2, R21.P$2, R23.P$2, U2.BUCK
- net GND: now also C4.P$2, C5.P$2, C6.P$2, C8.NEG, R12.P$1, R14.P$1, R16.P$1, R18.P$1, R20.P$1, R22.P$1, R24.P$1, R26.P$1, U2.FB_PRIM_D, U2.FB_PRIM_U, U2.GND, U2.PRIM
- net VBOOST: now also C3.P$1, U2.BOOST
Other:
- moved on the sheet: C2, C3, J1, L1, R10, R7, R8, R9, U2
